File: marauder_mini_pcb/marauder_mini_pcb.kicad_sch (KiCad schematic)
At the start: 8 parts, among them J1 Conn_01x10, SW1 SW_SPDT, U1 ESP32-WROOM-32

Commit message: Aggiornato circuito
Parts:
- J1: footprint Connector_PinHeader_2.54mm:PinHeader_1x10_P2.54mm_Vertical -> Library:PinHeader_1x10_P2.54mm_Vertical_largo
Connections:
- net GND: now also J1.8 (Pin_8); no longer D1.1 (K)
- net at C1.1, C2.1, R1.2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: now also SW1.1 (A); no longer SW1.2 (B)
- net at U1.26 (IO4): now also D1.1 (K)
- net at J1.10 (Pin_10): now also SW1.2 (B); no longer SW1.1 (A)
- no-connect marks 27 -> 26
Other:
- moved on the sheet: SW1
Changed lines of the file:
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@@
   (no_connect (at 77.47 93.98))
   (no_connect (at 107.95 109.22))
-  (no_connect (at 107.95 73.66))
   (no_connect (at 77.47 104.14))
   (no_connect (at 107.95 104.14))
@@
     (stroke (width 0) (type default))
   )
+  (wire (pts (xy 180.34 118.11) (xy 199.39 118.11))
+    (stroke (width 0) (type default))
+  )
   (wire (pts (xy 191.77 93.98) (xy 191.77 113.03))
     (stroke (width 0) (type default))
@@
     (stroke (width 0) (type default))
   )
+  (wire (pts (xy 204.47 67.31) (xy 204.47 73.66))
+    (stroke (width 0) (type default))
+  )
   (wire (pts (xy 161.29 99.06) (xy 161.29 104.14))
     (stroke (width 0) (type default))
@@
     (stroke (width 0) (type default))
   )
+  (wire (pts (xy 204.47 73.66) (xy 107.95 73.66))
+    (stroke (width 0) (type default))
+  )
   (wire (pts (xy 180.34 67.31) (xy 170.18 67.31))
     (stroke (width 0) (type default))
@@
   )
   (wire (pts (xy 107.95 66.04) (xy 132.08 66.04))
-    (stroke (width 0) (type default))
-  )
-  (wire (pts (xy 204.47 73.66) (xy 204.47 67.31))
     (stroke (width 0) (type default))
   )
@@
     )
   )
-  (symbol (lib_id "power:GND") (at 204.47 73.66 0) (unit 1)
-    (in_bom yes) (on_board yes) (dnp no) (fields_autoplaced)
-    (property "Reference" "#PWR04" (at 204.47 80.01 0)
-      (effects (font (size 1.27 1.27)) hide)
-    )
-    (property "Value" "GND" (at 204.47 78.74 0)
-      (effects (font (size 1.27 1.27)))
-    )
-    (property "Footprint" "" (at 204.47 73.66 0)
-      (effects (font (size 1.27 1.27)) hide)
-    )
-    (property "Datasheet" "" (at 204.47 73.66 0)
-      (effects (font (size 1.27 1.27)) hide)
-    )
-    (pin "1")
-    (instances
-      (project "marauder_mini_pcb"
-        (path "/d897c174-e854-4e44-8637-990dd2dbad11"
-          (reference "#PWR04") (unit 1)
+  (symbol (lib_id "power:GND") (at 180.34 118.11 270) (unit 1)
+    (in_bom yes) (on_board yes) (dnp no) (fields_autoplaced)
+    (property "Reference" "#PWR06" (at 173.99 118.11 0)
+      (effects (font (size 1.27 1.27)) hide)
+    )
+    (property "Value" "GND" (at 176.53 118.745 90)
+      (effects (font (size 1.27 1.27)) (justify right))
+    )
+    (property "Footprint" "" (at 180.34 118.11 0)
+      (effects (font (size 1.27 1.27)) hide)
+    )
+    (property "Datasheet" "" (at 180.34 118.11 0)
+      (effects (font (size 1.27 1.27)) hide)
+    )
+    (pin "1")
+    (instances
+      (project "marauder_mini_pcb"
+        (path "/d897c174-e854-4e44-8637-990dd2dbad11"
+          (reference "#PWR06") (unit 1)
         )
       )
@@
       (effects (font (size 1.27 1.27)) (justify left))
     )
-    (property "Footprint" "Connector_PinHeader_2.54mm:PinHeader_1x10_P2.54mm_Vertical" (at 204.47 125.73 0)
+    (property "Footprint" "Library:PinHeader_1x10_P2.54mm_Vertical_largo" (at 204.47 125.73 0)
       (effects (font (size 1.27 1.27)) hide)
     )
@@
     )
   )
-  (symbol (lib_id "Switch:SW_SPDT") (at 180.34 96.52 0) (unit 1)
-    (in_bom yes) (on_board yes) (dnp no) (fields_autoplaced)
-    (property "Reference" "SW1" (at 180.34 90.17 0)
+  (symbol (lib_id "Switch:SW_SPDT") (at 180.34 93.98 180) (unit 1)
+    (in_bom yes) (on_board yes) (dnp no) (fields_autoplaced)
+    (property "Reference" "SW1" (at 180.34 87.63 0)
       (effects (font (size 1.27 1.27)))
     )
-    (property "Value" "SW_SPDT" (at 180.34 92.71 0)
+    (property "Value" "SW_SPDT" (at 180.34 90.17 0)
       (effects (font (size 1.27 1.27)))
     )
-    (property "Footprint" "Button_Switch_SMD:SW_SPDT_PCM12" (at 180.34 96.52 0)
-      (effects (font (size 1.27 1.27)) hide)
-    )
-    (property "Datasheet" "~" (at 180.34 96.52 0)
-      (effects (font (size 1.27 1.27)) hide)
-    )
+    (property "Footprint" "Button_Switch_SMD:SW_SPDT_PCM12" (at 180.34 93.98 0)
+      (effects (font (size 1.27 1.27)) hide)
+    )
+    (property "Datasheet" "~" (at 180.34 93.98 0)
+      (effects (font (size 1.27 1.27)) hide)
+    )
