File: cc1101_pcb/cc1101_pcb.kicad_pcb (KiCad board)
At the start: 2 copper layers, 24 x 18.4 mm, 7 parts, among them J2 Conn_01x08_MountingPin, J3 Conn_02x04_Odd_Even_Shielded

Commit message: Aggiunta immagine settings arduino ide e aggiornate pcbs
Parts:
- added J1: Conn_01x08_MountingPin, Connector_PinHeader_2.54mm:PinHeader_1x08_P2.54mm_Vertical, B.Cu at (55.2, 78.9)
- J2: moved to B.Cu
- moved R1 13.4 mm to (41.6, 83.0)
- moved C2 12.8 mm to (41.7, 85.4), turned to 0 degrees
- moved C1 8.98 mm to (41.7, 87.8), turned to 0 degrees
- moved MCP1700 3.22 mm to (41.5, 91.4)
- moved LED 2.54 mm to (55.4, 83.2), turned to 180 degrees
- turned J2 to -90 degrees
Routing:
- net Net-(J1-Pin_2): track 8.78 -> 43.1 mm
- net Net-(J1-Pin_3): track 9.56 -> 38.1 mm, vias 1 -> 2
- net Net-(J1-Pin_4): track 13.9 -> 38.9 mm, vias 0 -> 1
- net Net-(J1-Pin_1): track 9.66 -> 30.3 mm, vias 0 -> 1
- net Net-(J1-Pin_5): track 18.6 -> 38.9 mm
- net Net-(J3-Pin_2): track 25.5 -> 11.0 mm
- net Net-(J1-Pin_6): track 20.4 -> 32.6 mm
- net Net-(D1-A): track 4.52 -> 11.6 mm
- net GND: track 0.00 -> 0.70 mm, vias 0 -> 2
Other:
- board size 24 x 18.4 mm -> 24 x 22 mm
