File: cc1101_pcb/cc1101_pcb.kicad_sch (KiCad schematic)
At the start: 7 parts, among them J2 Conn_01x08_MountingPin, J3 Conn_02x04_Odd_Even_Shielded, U1 MCP1700x-330xxTT

Commit message: Aggiunta immagine settings arduino ide e aggiornate pcbs
Parts:
- added J1: Conn_01x08_MountingPin, Connector_PinHeader_2.54mm:PinHeader_1x08_P2.54mm_Vertical, symbol Connector_Generic_MountingPin:Conn_01x08_MountingPin
Connections:
- net GND: now also J1.8 (Pin_8)
- net at J2.6 (Pin_6), J3.3 (Pin_3): now also J1.6 (Pin_6)
- net at J2.4 (Pin_4), J3.4 (Pin_4): now also J1.4 (Pin_4)
- net at J2.5 (Pin_5), J3.5 (Pin_5): now also J1.5 (Pin_5)
- net at J2.2 (Pin_2), J3.6 (Pin_6): now also J1.2 (Pin_2)
- net at J2.3 (Pin_3), J3.7 (Pin_7): now also J1.3 (Pin_3)
- net at J2.1 (Pin_1), U1.3 (VI): now also J1.1 (Pin_1)
- no-connect marks 4 -> 5
Other:
- moved on the sheet: J2
Changed lines of the file:
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@@
 (kicad_sch (version 20230121) (generator eeschema)
   (paper "A4")
+  (junction (at 111.76 128.27) (diameter 0) (color 0 0 0 0)
+  )
   (junction (at 106.68 74.93) (diameter 0) (color 0 0 0 0)
   )
+  (junction (at 109.22 125.73) (diameter 0) (color 0 0 0 0)
+  )
+  (junction (at 116.84 133.35) (diameter 0) (color 0 0 0 0)
+  )
   (junction (at 111.76 86.36) (diameter 0) (color 0 0 0 0)
   )
+  (junction (at 121.92 138.43) (diameter 0) (color 0 0 0 0)
+  )
+  (junction (at 104.14 120.65) (diameter 0) (color 0 0 0 0)
+  )
+  (junction (at 114.3 130.81) (diameter 0) (color 0 0 0 0)
+  )
+  (junction (at 106.68 123.19) (diameter 0) (color 0 0 0 0)
+  )
   (junction (at 118.11 59.69) (diameter 0) (color 0 0 0 0)
   )
-  (no_connect (at 119.38 113.03))
+  (no_connect (at 119.38 140.97))
   (no_connect (at 143.51 81.28))
   (no_connect (at 137.16 86.36))
-  (no_connect (at 127 118.11))
+  (no_connect (at 127 146.05))
+  (no_connect (at 93.98 135.89))
   (wire (pts (xy 130.81 73.66) (xy 125.73 73.66))
     (stroke (width 0) (type default))
@@
     (stroke (width 0) (type default))
   )
+  (wire (pts (xy 93.98 128.27) (xy 111.76 128.27))
+    (stroke (width 0) (type default))
+  )
   (wire (pts (xy 111.76 86.36) (xy 116.84 86.36))
     (stroke (width 0) (type default))
@@
     (stroke (width 0) (type default))
   )
+  (wire (pts (xy 104.14 120.65) (xy 104.14 140.97))
+    (stroke (width 0) (type default))
+  )
   (wire (pts (xy 111.76 86.36) (xy 111.76 88.9))
     (stroke (width 0) (type default))
@@
     (stroke (width 0) (type default))
   )
-  (wire (pts (xy 106.68 113.03) (xy 106.68 100.33))
+  (wire (pts (xy 106.68 140.97) (xy 106.68 123.19))
     (stroke (width 0) (type default))
   )
@@
     (stroke (width 0) (type default))
   )
-  (wire (pts (xy 121.92 113.03) (xy 121.92 111.76))
-    (stroke (width 0) (type default))
-  )
-  (wire (pts (xy 116.84 113.03) (xy 116.84 91.44))
+  (wire (pts (xy 93.98 133.35) (xy 116.84 133.35))
+    (stroke (width 0) (type default))
+  )
+  (wire (pts (xy 121.92 140.97) (xy 121.92 138.43))
+    (stroke (width 0) (type default))
+  )
+  (wire (pts (xy 106.68 123.19) (xy 106.68 100.33))
+    (stroke (width 0) (type default))
+  )
+  (wire (pts (xy 116.84 140.97) (xy 116.84 133.35))
     (stroke (width 0) (type default))
   )
@@
     (stroke (width 0) (type default))
   )
-  (wire (pts (xy 114.3 107.95) (xy 114.3 113.03))
-    (stroke (width 0) (type default))
-  )
-  (wire (pts (xy 104.14 95.25) (xy 104.14 113.03))
+  (wire (pts (xy 114.3 107.95) (xy 114.3 130.81))
+    (stroke (width 0) (type default))
+  )
+  (wire (pts (xy 104.14 95.25) (xy 104.14 120.65))
     (stroke (width 0) (type default))
   )
@@
     (stroke (width 0) (type default))
   )
+  (wire (pts (xy 93.98 120.65) (xy 104.14 120.65))
+    (stroke (width 0) (type default))
+  )
+  (wire (pts (xy 93.98 130.81) (xy 114.3 130.81))
+    (stroke (width 0) (type default))
+  )
   (wire (pts (xy 116.84 91.44) (xy 127 91.44))
     (stroke (width 0) (type default))
@@
     (stroke (width 0) (type default))
   )
+  (wire (pts (xy 116.84 133.35) (xy 116.84 91.44))
+    (stroke (width 0) (type default))
+  )
+  (wire (pts (xy 93.98 123.19) (xy 106.68 123.19))
+    (stroke (width 0) (type default))
+  )
+  (wire (pts (xy 111.76 128.27) (xy 111.76 104.14))
+    (stroke (width 0) (type default))
+  )
   (wire (pts (xy 116.84 74.93) (xy 106.68 74.93))
     (stroke (width 0) (type default))
@@
     (stroke (width 0) (type default))
   )
+  (wire (pts (xy 93.98 125.73) (xy 109.22 125.73))
+    (stroke (width 0) (type default))
+  )
   (wire (pts (xy 106.68 74.93) (xy 106.68 78.74))
     (stroke (width 0) (type default))
@@
     (stroke (width 0) (type default))
   )
-  (wire (pts (xy 109.22 96.52) (xy 109.22 113.03))
+  (wire (pts (xy 114.3 130.81) (xy 114.3 140.97))
+    (stroke (width 0) (type default))
+  )
+  (wire (pts (xy 109.22 96.52) (xy 109.22 125.73))
     (stroke (width 0) (type default))
   )
@@
     (stroke (width 0) (type default))
   )
+  (wire (pts (xy 121.92 138.43) (xy 121.92 111.76))
+    (stroke (width 0) (type default))
+  )
   (wire (pts (xy 95.25 74.93) (xy 106.68 74.93))
     (stroke (width 0) (type default))
@@
     (stroke (width 0) (type default))
   )
-  (wire (pts (xy 111.76 113.03) (xy 111.76 104.14))
+  (wire (pts (xy 111.76 140.97) (xy 111.76 128.27))
+    (stroke (width 0) (type default))
+  )
+  (wire (pts (xy 109.22 125.73) (xy 109.22 140.97))
+    (stroke (width 0) (type default))
+  )
+  (wire (pts (xy 93.98 138.43) (xy 121.92 138.43))
     (stroke (width 0) (type default))
   )
@@
     )
   )
+  (symbol (lib_id "Connector_Generic_MountingPin:Conn_01x08_MountingPin") (at 88.9 128.27 0) (mirror y) (unit 1)
+    (in_bom yes) (on_board yes) (dnp no)
+    (property "Reference" "J1" (at 83.82 129.8956 90)
+      (effects (font (size 1.27 1.27)))
+    )
+    (property "Value" "Conn_01x08_MountingPin" (at 86.36 129.8956 90)
+      (effects (font (size 1.27 1.27)))
+    )
+    (property "Footprint" "Connector_PinHeader_2.54mm:PinHeader_1x08_P2.54mm_Vertical" (at 88.9 128.27 0)
+      (effects (font (size 1.27 1.27)) hide)
+    )
+    (property "Datasheet" "~" (at 88.9 128.27 0)
+      (effects (font (size 1.27 1.27)) hide)
+    )
+    (pin "1")
+    (pin "2")
+    (pin "3")
+    (pin "4")
+    (pin "5")
+    (pin "6")
+    (pin "7")
+    (pin "8")
+    (pin "MP")
+    (instances
+      (project "cc1101_pcb"
+        (path "/ad378880-11bf-499d-a2ba-9010a6a5b21b"
+          (reference "J1") (unit 1)
+        )
+      )
+    )
+  )
   (symbol (lib_id "power:GND") (at 133.35 111.76 90) (unit 1)
     (in_bom yes) (on_board yes) (dnp no) (fields_autoplaced)
@@
     )
   )
-  (symbol (lib_id "Connector_Generic_MountingPin:Conn_01x08_MountingPin") (at 111.76 118.11 90) (mirror x) (unit 1)
+  (symbol (lib_id "Connector_Generic_MountingPin:Conn_01x08_MountingPin") (at 111.76 146.05 90) (mirror x) (unit 1)
     (in_bom yes) (on_board yes) (dnp no)
-    (property "Reference" "J2" (at 113.3856 123.19 90)
-      (effects (font (size 1.27 1.27)))
-    )
-    (property "Value" "Conn_01x08_MountingPin" (at 113.3856 120.65 90)
-      (effects (font (size 1.27 1.27)))
-    )
-    (property "Footprint" "Connector_PinHeader_2.54mm:PinHeader_1x08_P2.54mm_Vertical" (at 111.76 118.11 0)
-      (effects (font (size 1.27 1.27)) hide)
-    )
-    (property "Datasheet" "~" (at 111.76 118.11 0)
-      (effects (font (size 1.27 1.27)) hide)
-    )
+    (property "Reference" "J2" (at 113.3856 151.13 90)
+      (effects (font (size 1.27 1.27)))
+    )
+    (property "Value" "Conn_01x08_MountingPin" (at 113.3856 148.59 90)
+      (effects (font (size 1.27 1.27)))
+    )
+    (property "Footprint" "Connector_PinHeader_2.54mm:PinHeader_1x08_P2.54mm_Vertical" (at 111.76 146.05 0)
+      (effects (font (size 1.27 1.27)) hide)
+    )
+    (property "Datasheet" "~" (at 111.76 146.05 0)
+      (effects (font (size 1.27 1.27)) hide)
+    )
