File: marauder_mini_pcb_2/marauder_mini_pcb.kicad_pcb (KiCad board)
At the start: 2 copper layers, 37 x 20 mm, 9 parts, among them J1 Conn_01x10, SW1 SW_SPDT, SW2 SW_Push, SW3 SW_Push, U1 ESP32-WROOM-32

Commit message: Modifiche varie che non voglio controllare
Changed lines of the file:
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@@
       (drillshape 0)
       (scaleselection 1)
-      (outputdirectory "")
+      (outputdirectory "GERBER/")
     )
   )
@@
     (fp_line (start 1 0.625) (end 1 -0.625)
       (stroke (width 0.1) (type solid)) (layer "B.Fab"))
-    (pad "1" smd roundrect (at -1.0375 0 180) (size 1.175 1.45) (layers "B.Cu" "B.Paste" "B.Mask") (roundrect_rratio 0.212766)
+    (pad "1" smd roundrect (at -1.0375 0 180) (size 1.175 1.45) (layers "B.Cu" "B.Paste" "B.Mask") (roundrect_rratio 0.2127659574)
       (net 1 "GND") (pinfunction "K") (pintype "passive"))
-    (pad "2" smd roundrect (at 1.0375 0 180) (size 1.175 1.45) (layers "B.Cu" "B.Paste" "B.Mask") (roundrect_rratio 0.212766)
+    (pad "2" smd roundrect (at 1.0375 0 180) (size 1.175 1.45) (layers "B.Cu" "B.Paste" "B.Mask") (roundrect_rratio 0.2127659574)
       (net 2 "Net-(D1-A)") (pinfunction "A") (pintype "passive"))
     (model "${KICAD6_3DMODEL_DIR}/Capacitor_SMD.3dshapes/C_0805_2012Metric.wrl"
@@
     (fp_line (start 1 0.625) (end 1 -0.625)
       (stroke (width 0.1) (type solid)) (layer "B.Fab"))
-    (pad "1" smd roundrect (at -1.0375 0 180) (size 1.175 1.45) (layers "B.Cu" "B.Paste" "B.Mask") (roundrect_rratio 0.212766)
+    (pad "1" smd roundrect (at -1.0375 0 180) (size 1.175 1.45) (layers "B.Cu" "B.Paste" "B.Mask") (roundrect_rratio 0.2127659574)
       (net 39 "Net-(SW1-A)") (pintype "passive"))
-    (pad "2" smd roundrect (at 1.0375 0 180) (size 1.175 1.45) (layers "B.Cu" "B.Paste" "B.Mask") (roundrect_rratio 0.212766)
+    (pad "2" smd roundrect (at 1.0375 0 180) (size 1.175 1.45) (layers "B.Cu" "B.Paste" "B.Mask") (roundrect_rratio 0.2127659574)
       (net 1 "GND") (pintype "passive"))
     (model "${KICAD6_3DMODEL_DIR}/Capacitor_SMD.3dshapes/C_0805_2012Metric.wrl"
@@
     (fp_line (start 1 0.625) (end 1 -0.625)
       (stroke (width 0.1) (type solid)) (layer "B.Fab"))
-    (pad "1" smd roundrect (at -1.0375 0) (size 1.175 1.45) (layers "B.Cu" "B.Paste" "B.Mask") (roundrect_rratio 0.212766)
+    (pad "1" smd roundrect (at -1.0375 0) (size 1.175 1.45) (layers "B.Cu" "B.Paste" "B.Mask") (roundrect_rratio 0.2127659574)
       (net 39 "Net-(SW1-A)") (pintype "passive"))
-    (pad "2" smd roundrect (at 1.0375 0) (size 1.175 1.45) (layers "B.Cu" "B.Paste" "B.Mask") (roundrect_rratio 0.212766)
+    (pad "2" smd roundrect (at 1.0375 0) (size 1.175 1.45) (layers "B.Cu" "B.Paste" "B.Mask") (roundrect_rratio 0.2127659574)
       (net 1 "GND") (pintype "passive"))
     (model "${KICAD6_3DMODEL_DIR}/Capacitor_SMD.3dshapes/C_0805_2012Metric.wrl"
@@
     (fp_line (start 1 0.625) (end 1 -0.625)
       (stroke (width 0.1) (type solid)) (layer "B.Fab"))
-    (pad "1" smd roundrect (at -1.0375 0 180) (size 1.175 1.45) (layers "B.Cu" "B.Paste" "B.Mask") (roundrect_rratio 0.212766)
+    (pad "1" smd roundrect (at -1.0375 0 180) (size 1.175 1.45) (layers "B.Cu" "B.Paste" "B.Mask") (roundrect_rratio 0.2127659574)
       (net 2 "Net-(D1-A)") (pintype "passive"))
-    (pad "2" smd roundrect (at 1.0375 0 180) (size 1.175 1.45) (layers "B.Cu" "B.Paste" "B.Mask") (roundrect_rratio 0.212766)
+    (pad "2" smd roundrect (at 1.0375 0 180) (size 1.175 1.45) (layers "B.Cu" "B.Paste" "B.Mask") (roundrect_rratio 0.2127659574)
       (net 39 "Net-(SW1-A)") (pintype "passive"))
     (model "${KICAD6_3DMODEL_DIR}/Capacitor_SMD.3dshapes/C_0805_2012Metric.wrl"
@@
     (effects (font (size 1.5 1.5) (thickness 0.17)) (justify left bottom))
   )
+  (dimension (type aligned) (layer "User.2")
+    (pts (xy 87 54.5) (xy 50 54.5))
+    (height -27)
+    (gr_text "37,0000 mm" (at 68.5 80.35) (layer "User.2")
+      (effects (font (size 1 1) (thickness 0.15)))
+    )
+    (format (prefix "") (suffix "") (units 3) (units_format 1) (precision 4))
+    (style (thickness 0.15) (arrow_length 1.27) (text_position_mode 0) (extension_height 0.58642) (extension_offset 0.5) keep_text_aligned)
+  )
+  (dimension (type aligned) (layer "User.2")
+    (pts (xy 50 70) (xy 50 50))
+    (height -9)
+    (gr_text "20,0000 mm" (at 39.85 60 90) (layer "User.2")
+      (effects (font (size 1 1) (thickness 0.15)))
+    )
+    (format (prefix "") (suffix "") (units 3) (units_format 1) (precision 4))
+    (style (thickness 0.15) (arrow_length 1.27) (text_position_mode 0) (extension_height 0.58642) (extension_offset 0.5) keep_text_aligned)
+  )
   (via (at 62.3 55.3) (size 0.8) (drill 0.4) (layers "F.Cu" "B.Cu") (free) (net 1))

Commit message: Aggiornato marauder e pcb
Parts:
- added R2: 10K, Capacitor_SMD:C_0805_2012Metric_Pad1.18x1.45mm_HandSolder, B.Cu at (62.6, 55.1)
- renumbered LED to D1
Routing:
- net Net-(U1-EN): track 7.19 -> 9.96 mm
- net Net-(SW1-A): track 33.1 -> 34.3 mm
Changed lines of the file:
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@@
     (property "ki_keywords" "LED diode")
     (attr smd)
-    (fp_text reference "LED" (at 0.0375 -1.6) (layer "B.SilkS")
+    (fp_text reference "D1" (at 0.0375 -1.6) (layer "B.SilkS")
         (effects (font (size 1 1) (thickness 0.15)) (justify mirror))
     )
@@
       (net 38 "unconnected-(SW1-C-Pad3)") (pinfunction "C") (pintype "passive"))
     (model "${KICAD6_3DMODEL_DIR}/Button_Switch_SMD.3dshapes/SW_SPDT_PCM12.wrl"
+      (offset (xyz 0 0 0))
+      (scale (xyz 1 1 1))
+      (rotate (xyz 0 0 0))
+    )
+  )
+  (footprint "Capacitor_SMD:C_0805_2012Metric_Pad1.18x1.45mm_HandSolder" (layer "B.Cu")
+    (at 62.5575 55.11)
+    (descr "Capacitor SMD 0805 (2012 Metric), square (rectangular) end terminal, IPC_7351 nominal with elongated pad for handsoldering. (Body size source: IPC-SM-782 page 76, https://www.pcb-3d.com/wordpress/wp-content/uploads/ipc-sm-782a_amendment_1_and_2.pdf, https://docs.google.com/spreadsheets/d/1BsfQQcO9C6DZCsRaXUlFlo91Tg2WpOkGARC1WS5S8t0/edit?usp=sharing), generated with kicad-footprint-generator")
+    (tags "capacitor handsolder")
+    (property "Sheetfile" "marauder_mini_pcb.kicad_sch")
+    (property "Sheetname" "")
+    (property "ki_description" "Resistor")
+    (property "ki_keywords" "R res resistor")
+    (attr smd)
+    (fp_text reference "R2" (at -0.0075 -1.62) (layer "B.SilkS")
+        (effects (font (size 1 1) (thickness 0.15)) (justify mirror))
+    )
+    (fp_text value "10K" (at 0 -1.68) (layer "B.Fab") hide
+        (effects (font (size 1 1) (thickness 0.15)) (justify mirror))
+    )
+    (fp_text user "${REFERENCE}" (at 0 0) (layer "B.Fab")
+        (effects (font (size 0.5 0.5) (thickness 0.08)) (justify mirror))
+    )
+    (fp_line (start -0.261252 -0.735) (end 0.261252 -0.735)
+      (stroke (width 0.12) (type solid)) (layer "B.SilkS"))
+    (fp_line (start -0.261252 0.735) (end 0.261252 0.735)
+      (stroke (width 0.12) (type solid)) (layer "B.SilkS"))
+    (fp_line (start -1.88 -0.98) (end -1.88 0.98)
+      (stroke (width 0.05) (type solid)) (layer "B.CrtYd"))
+    (fp_line (start -1.88 0.98) (end 1.88 0.98)
+      (stroke (width 0.05) (type solid)) (layer "B.CrtYd"))
+    (fp_line (start 1.88 -0.98) (end -1.88 -0.98)
+      (stroke (width 0.05) (type solid)) (layer "B.CrtYd"))
+    (fp_line (start 1.88 0.98) (end 1.88 -0.98)
+      (stroke (width 0.05) (type solid)) (layer "B.CrtYd"))
+    (fp_line (start -1 -0.625) (end -1 0.625)
+      (stroke (width 0.1) (type solid)) (layer "B.Fab"))
+    (fp_line (start -1 0.625) (end 1 0.625)
+      (stroke (width 0.1) (type solid)) (layer "B.Fab"))
+    (fp_line (start 1 -0.625) (end -1 -0.625)
+      (stroke (width 0.1) (type solid)) (layer "B.Fab"))
+    (fp_line (start 1 0.625) (end 1 -0.625)
+      (stroke (width 0.1) (type solid)) (layer "B.Fab"))
+    (pad "1" smd roundrect (at -1.0375 0) (size 1.175 1.45) (layers "B.Cu" "B.Paste" "B.Mask") (roundrect_rratio 0.212766)
+      (net 39 "Net-(SW1-A)") (pintype "passive"))
+    (pad "2" smd roundrect (at 1.0375 0) (size 1.175 1.45) (layers "B.Cu" "B.Paste" "B.Mask") (roundrect_rratio 0.212766)
+      (net 42 "Net-(U1-EN)") (pintype "passive"))
+    (model "${KICAD6_3DMODEL_DIR}/Capacitor_SMD.3dshapes/C_0805_2012Metric.wrl"
       (offset (xyz 0 0 0))
       (scale (xyz 1 1 1))
@@
   (segment (start 57.325 54.675) (end 57.325 55.1) (width 0.3) (layer "B.Cu") (net 39))
   (segment (start 55.2 55.1) (end 57.325 55.1) (width 0.3) (layer "B.Cu") (net 39))
+  (segment (start 67.2 53.9) (end 61.52 53.9) (width 0.3) (layer "B.Cu") (net 39))
   (segment (start 58.1 53.9) (end 57.325 54.675) (width 0.3) (layer "B.Cu") (net 39))
   (segment (start 55.2 58.6) (end 55.2 55.1) (width 0.3) (layer "B.Cu") (net 39))
@@
   (segment (start 57.6 61) (end 55.2 58.6) (width 0.3) (layer "B.Cu") (net 39))
   (segment (start 61.425 66.925) (end 61.425 67.7) (width 0.3) (layer "B.Cu") (net 39))
-  (segment (start 67.2 53.9) (end 58.1 53.9) (width 0.3) (layer "B.Cu") (net 39))
+  (segment (start 61.52 53.9) (end 58.1 53.9) (width 0.3) (layer "B.Cu") (net 39))
   (segment (start 57.6 64.54) (end 59.04 64.54) (width 0.3) (layer "B.Cu") (net 39))
   (segment (start 59.04 64.54) (end 61.425 66.925) (width 0.3) (layer "B.Cu") (net 39))
+  (segment (start 61.52 55.11) (end 61.52 53.9) (width 0.25) (layer "B.Cu") (net 39))
   (segment (start 57.25 66.34) (end 57.34 66.25) (width 0.3) (layer "B.Cu") (net 39))
   (segment (start 55 63.7) (end 52.335 66.365) (width 0.25) (layer "F.Cu") (net 41))
@@
   (segment (start 66.3 55.4) (end 66.3 51.255) (width 0.25) (layer "F.Cu") (net 42))
   (via (at 66.2 55.5) (size 0.8) (drill 0.4) (layers "F.Cu" "B.Cu") (free) (net 42))
+  (segment (start 63.595 55.11) (end 65.81 55.11) (width 0.25) (layer "B.Cu") (net 42))
   (segment (start 66.2 58.4) (end 66.2 55.5) (width 0.25) (layer "B.Cu") (net 42))
+  (segment (start 65.81 55.11) (end 66.2 55.5) (width 0.25) (layer "B.Cu") (net 42))
   (zone (net 1) (net_name "GND") (layers "F&B.Cu") (hatch edge 0.5)
     (connect_pads yes (clearance 0.6))
