File: marauder_mini_pcb_2/marauder_mini_pcb.kicad_sch (KiCad schematic)
At the start: 9 parts, among them J1 Conn_01x10, SW1 SW_SPDT, SW2 SW_Push, SW3 SW_Push, U1 ESP32-WROOM-32

Commit message: Aggiornato marauder e pcb
Parts:
- added R2: 10K, Capacitor_SMD:C_0805_2012Metric_Pad1.18x1.45mm_HandSolder, symbol Device:R
Connections:
- net at C1.1, C2.1, R1.2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: now also R2.1
- net at SW3.2, U1.3 (EN): now also R2.2
Changed lines of the file:
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@@
 (kicad_sch (version 20230121) (generator eeschema)
   (paper "A4")
+  (junction (at 63.5 63.5) (diameter 0) (color 0 0 0 0)
+  )
   (junction (at 153.67 104.14) (diameter 0) (color 0 0 0 0)
   )
@@
   )
   (junction (at 161.29 91.44) (diameter 0) (color 0 0 0 0)
+  )
+  (junction (at 92.71 53.34) (diameter 0) (color 0 0 0 0)
   )
   (no_connect (at 77.47 71.12))
@@
     (stroke (width 0) (type default))
   )
-  (wire (pts (xy 92.71 58.42) (xy 92.71 49.53))
+  (wire (pts (xy 92.71 58.42) (xy 92.71 53.34))
+    (stroke (width 0) (type default))
+  )
+  (wire (pts (xy 92.71 53.34) (xy 92.71 49.53))
     (stroke (width 0) (type default))
   )
@@
     (stroke (width 0) (type default))
   )
+  (wire (pts (xy 63.5 63.5) (xy 77.47 63.5))
+    (stroke (width 0) (type default))
+  )
   (wire (pts (xy 191.77 93.98) (xy 191.77 113.03))
     (stroke (width 0) (type default))
   )
+  (wire (pts (xy 71.12 53.34) (xy 63.5 53.34))
+    (stroke (width 0) (type default))
+  )
   (wire (pts (xy 185.42 93.98) (xy 191.77 93.98))
     (stroke (width 0) (type default))
@@
     (stroke (width 0) (type default))
   )
+  (wire (pts (xy 63.5 53.34) (xy 63.5 63.5))
+    (stroke (width 0) (type default))
+  )
   (wire (pts (xy 151.13 63.5) (xy 151.13 52.07))
     (stroke (width 0) (type default))
@@
     (stroke (width 0) (type default))
   )
+  (wire (pts (xy 78.74 53.34) (xy 92.71 53.34))
+    (stroke (width 0) (type default))
+  )
   (wire (pts (xy 199.39 128.27) (xy 121.92 128.27))
     (stroke (width 0) (type default))
@@
     (stroke (width 0) (type default))
   )
-  (wire (pts (xy 57.15 63.5) (xy 77.47 63.5))
+  (wire (pts (xy 57.15 63.5) (xy 63.5 63.5))
     (stroke (width 0) (type default))
   )
@@
     )
   )
+  (symbol (lib_id "Device:R") (at 74.93 53.34 270) (unit 1)
+    (in_bom yes) (on_board yes) (dnp no) (fields_autoplaced)
+    (property "Reference" "R2" (at 74.93 46.99 90)
+      (effects (font (size 1.27 1.27)))
+    )
+    (property "Value" "10K" (at 74.93 49.53 90)
+      (effects (font (size 1.27 1.27)))
+    )
+    (property "Footprint" "Capacitor_SMD:C_0805_2012Metric_Pad1.18x1.45mm_HandSolder" (at 74.93 51.562 90)
+      (effects (font (size 1.27 1.27)) hide)
+    )
+    (property "Datasheet" "~" (at 74.93 53.34 0)
+      (effects (font (size 1.27 1.27)) hide)
+    )
+    (pin "1")
+    (pin "2")
+    (instances
+      (project "marauder_mini_pcb"
+        (path "/d897c174-e854-4e44-8637-990dd2dbad11"
+          (reference "R2") (unit 1)
+        )
+      )
+    )
+  )
   (symbol (lib_id "power:GND") (at 172.72 53.34 0) (unit 1)
     (in_bom yes) (on_board yes) (dnp no) (fields_autoplaced)
@@
   (symbol (lib_id "Device:R") (at 184.15 67.31 270) (unit 1)
     (in_bom yes) (on_board yes) (dnp no) (fields_autoplaced)
-    (property "Reference" "R1" (at 184.15 72.39 90)
-      (effects (font (size 1.27 1.27)))
-    )
-    (property "Value" "R" (at 184.15 69.85 90)
+    (property "Reference" "R1" (at 184.15 60.96 90)
+      (effects (font (size 1.27 1.27)))
+    )
+    (property "Value" "R" (at 184.15 63.5 90)
       (effects (font (size 1.27 1.27)))
     )
     (property "Footprint" "Capacitor_SMD:C_0805_2012Metric_Pad1.18x1.45mm_HandSolder" (at 184.15 65.532 90)
-      (effects (font (size 1.27 1.27)))
+      (effects (font (size 1.27 1.27)) hide)
     )
     (property "Datasheet" "~" (at 184.15 67.31 0)
