File: marauder_mini_pcb_ext_antenna/marauder_mini_pcb.kicad_pcb (KiCad board)
At the start: 2 copper layers, 32.4 x 30.5 mm, 9 parts, among them J1 Conn_01x10, SW1 SW_SPDT, U1 ESP32-WROOM-32

Commit message: Aggiornato marauder e pcb
Parts:
- added R2: 10k, Capacitor_SMD:C_0805_2012Metric_Pad1.18x1.45mm_HandSolder, B.Cu at (80.2, 59.8)
- renumbered LED to D1, IO0 to SW2, EN to SW3
Routing:
- net Net-(U1-EN): track 35.1 -> 35.8 mm
Other:
- board size 32.4 x 30.5 mm -> 32.5 x 25 mm
- board text added: "Flipper ESP32 V2.1"
- board text removed: "Flipper ESP32 V2"
