File: marauder_mini_pcb_ext_antenna/marauder_mini_pcb.kicad_sch (KiCad schematic)
At the start: 9 parts, among them J1 Conn_01x10, SW1 SW_SPDT, SW2 SW_Push, SW3 SW_Push, U1 ESP32-WROOM-32

Commit message: Aggiornato marauder e pcb
Parts:
- added R2: 10k, Capacitor_SMD:C_0805_2012Metric_Pad1.18x1.45mm_HandSolder, symbol Device:R
Connections:
- net at C1.1, C2.1, R1.2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: now also R2.2
- net at SW3.2, U1.3 (EN): now also R2.1
Changed lines of the file:
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@@
 (kicad_sch (version 20230121) (generator eeschema)
   (paper "A4")
+  (junction (at 63.5 63.5) (diameter 0) (color 0 0 0 0)
+  )
   (junction (at 153.67 104.14) (diameter 0) (color 0 0 0 0)
   )
@@
   )
   (junction (at 146.05 91.44) (diameter 0) (color 0 0 0 0)
+  )
+  (junction (at 92.71 54.61) (diameter 0) (color 0 0 0 0)
   )
   (junction (at 161.29 91.44) (diameter 0) (color 0 0 0 0)
@@
     (stroke (width 0) (type default))
   )
+  (wire (pts (xy 92.71 54.61) (xy 92.71 49.53))
+    (stroke (width 0) (type default))
+  )
   (wire (pts (xy 118.11 130.81) (xy 199.39 130.81))
     (stroke (width 0) (type default))
@@
     (stroke (width 0) (type default))
   )
-  (wire (pts (xy 92.71 58.42) (xy 92.71 49.53))
+  (wire (pts (xy 92.71 58.42) (xy 92.71 54.61))
     (stroke (width 0) (type default))
   )
@@
     (stroke (width 0) (type default))
   )
+  (wire (pts (xy 63.5 63.5) (xy 77.47 63.5))
+    (stroke (width 0) (type default))
+  )
   (wire (pts (xy 199.39 67.31) (xy 204.47 67.31))
     (stroke (width 0) (type default))
@@
     (stroke (width 0) (type default))
   )
+  (wire (pts (xy 63.5 54.61) (xy 63.5 63.5))
+    (stroke (width 0) (type default))
+  )
   (wire (pts (xy 204.47 67.31) (xy 204.47 73.66))
     (stroke (width 0) (type default))
@@
     (stroke (width 0) (type default))
   )
+  (wire (pts (xy 67.31 54.61) (xy 63.5 54.61))
+    (stroke (width 0) (type default))
+  )
   (wire (pts (xy 128.27 71.12) (xy 107.95 71.12))
     (stroke (width 0) (type default))
@@
     (stroke (width 0) (type default))
   )
+  (wire (pts (xy 74.93 54.61) (xy 92.71 54.61))
+    (stroke (width 0) (type default))
+  )
   (wire (pts (xy 46.99 63.5) (xy 38.1 63.5))
     (stroke (width 0) (type default))
   )
-  (wire (pts (xy 57.15 63.5) (xy 77.47 63.5))
+  (wire (pts (xy 57.15 63.5) (xy 63.5 63.5))
     (stroke (width 0) (type default))
   )
@@
         )
       )
+    )
+  )
+  (symbol (lib_id "Device:R") (at 71.12 54.61 90) (unit 1)
+    (in_bom yes) (on_board yes) (dnp no) (fields_autoplaced)
+    (property "Reference" "R2" (at 71.12 48.26 90)
+      (effects (font (size 1.27 1.27)))
+    )
+    (property "Value" "10k" (at 71.12 50.8 90)
+      (effects (font (size 1.27 1.27)))
+    )
+    (property "Footprint" "Capacitor_SMD:C_0805_2012Metric_Pad1.18x1.45mm_HandSolder" (at 71.12 56.388 90)
+      (effects (font (size 1.27 1.27)) hide)
+    )
+    (property "Datasheet" "~" (at 71.12 54.61 0)
+      (effects (font (size 1.27 1.27)) hide)
+    )
+    (pin "1")
+    (pin "2")
+    (instances
+      (project "marauder_mini_pcb"
+        (path "/d897c174-e854-4e44-8637-990dd2dbad11"
+          (reference "R2") (unit 1)
+        )
+      )
